File: pcb/module.kicad_sch (KiCad schematic)
At the start: 19 parts

Commit message: 100nf decoupling caps
Parts:
- removed C3: 100uF, symbol Device:C
Changed lines of the file:
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@@
-	)
-	(junction
-		(at 62.23 186.69)
-		(diameter 0)
-		(color 0 0 0 0)
 	)
 	(junction
@@
 		(color 0 0 0 0)
 	)
-	(junction
-		(at 54.61 186.69)
-		(diameter 0)
-		(color 0 0 0 0)
-	)
 	(wire
 		(pts
@@
 	(wire
 		(pts
-			(xy 62.23 176.53) (xy 62.23 186.69)
+			(xy 62.23 176.53) (xy 62.23 182.88)
 		)
 		(stroke
@@
 	(wire
 		(pts
-			(xy 54.61 176.53) (xy 54.61 186.69)
-		)
-		(stroke
-			(width 0)
-			(type default)
-		)
-	)
-	(wire
-		(pts
-			(xy 62.23 186.69) (xy 62.23 190.5)
-		)
-		(stroke
-			(width 0)
-			(type default)
-		)
-	)
-	(wire
-		(pts
-			(xy 54.61 186.69) (xy 54.61 190.5)
+			(xy 54.61 176.53) (xy 54.61 182.88)
 		)
 		(stroke
@@
 	(symbol
 		(lib_id "power:+5V")
-		(at 62.23 190.5 180)
+		(at 62.23 182.88 180)
 		(unit 1)
 		(exclude_from_sim no)
@@
 		(dnp no)
 		(property "Reference" "#PWR?"
-			(at 62.23 186.69 0)
+			(at 62.23 179.07 0)
 			(effects
 				(font
@@
 		)
 		(property "Value" "+5V"
-			(at 63.5 195.072 0)
+			(at 63.5 187.452 0)
 			(effects
 				(font
@@
 		)
 		(property "Footprint" ""
-			(at 62.23 190.5 0)
+			(at 62.23 182.88 0)
 			(effects
 				(font
@@
 		)
 		(property "Datasheet" ""
-			(at 62.23 190.5 0)
+			(at 62.23 182.88 0)
 			(effects
 				(font
@@
 		)
 		(property "Description" "Power symbol creates a global label with name \"+5V\""
-			(at 62.23 190.5 0)
+			(at 62.23 182.88 0)
 			(effects
 				(font
@@
 				(path "/be5c4baa-09c6-44d9-9a7a-613f890eb055/fd83976f-fb21-44bf-9e12-4fb0dd274971"
 					(reference "#PWR022")
-					(unit 1)
-				)
-			)
-		)
-	)
-	(symbol
-		(lib_id "Device:C")
-		(at 58.42 186.69 90)
-		(unit 1)
-		(exclude_from_sim no)
-		(in_bom yes)
-		(on_board yes)
-		(dnp no)
-		(property "Reference" "C3"
-			(at 58.42 183.388 90)
-			(effects
-				(font
-					(size 1.27 1.27)
-				)
-			)
-		)
-		(property "Value" "100uF"
-			(at 58.42 190.754 90)
-			(effects
-				(font
-					(size 1.27 1.27)
-				)
-			)
-		)
-		(property "Footprint" ""
-			(at 62.23 185.7248 0)
-			(effects
-				(font
-					(size 1.27 1.27)
-				)
-				(hide yes)
-			)
-		)
-		(property "Datasheet" "~"
-			(at 58.42 186.69 0)
-			(effects
-				(font
-					(size 1.27 1.27)
-				)
-				(hide yes)
-			)
-		)
-		(property "Description" "Unpolarized capacitor"
-			(at 58.42 186.69 0)
-			(effects
-				(font
-					(size 1.27 1.27)
-				)
-				(hide yes)
-			)
-		)
-		(pin "1"
-		)
-		(pin "2"
-		)
-		(instances
-			(project ""
-				(path "/be5c4baa-09c6-44d9-9a7a-613f890eb055/2999f972-2a97-404c-8e8a-f1944f7da9fa"
-					(reference "C16")
-					(unit 1)
-				)
-				(path "/be5c4baa-09c6-44d9-9a7a-613f890eb055/528ad272-0ccd-4592-bf87-7b929987564e"
-					(reference "C15")
-					(unit 1)
-				)
-				(path "/be5c4baa-09c6-44d9-9a7a-613f890eb055/67888a8a-5a99-4148-a7fe-b94d8037f0ce"
-					(reference "C19")
-					(unit 1)
-				)
-				(path "/be5c4baa-09c6-44d9-9a7a-613f890eb055/8028cfdb-12ff-4440-aacc-65120448082b"
-					(reference "C12")
-					(unit 1)
-				)
-				(path "/be5c4baa-09c6-44d9-9a7a-613f890eb055/9f234ac0-edf2-4a35-84a2-e161cf8af174"
-					(reference "C7")
-					(unit 1)
-				)
-				(path "/be5c4baa-09c6-44d9-9a7a-613f890eb055/b313231a-6784-4797-92a7-75ee8640b712"
-					(reference "C11")
-					(unit 1)
-				)
-				(path "/be5c4baa-09c6-44d9-9a7a-613f890eb055/c204a1f2-0e4b-4d6c-acfd-a7f0c358d49c"
-					(reference "C5")
-					(unit 1)
-				)
-				(path "/be5c4baa-09c6-44d9-9a7a-613f890eb055/c92745bd-27fd-4104-92b5-8f961dfa3137"
-					(reference "C3")
-					(unit 1)
-				)
-				(path "/be5c4baa-09c6-44d9-9a7a-613f890eb055/fd83976f-fb21-44bf-9e12-4fb0dd274971"
-					(reference "C8")
 					(unit 1)
 				)
@@
 	(symbol
 		(lib_id "power:GND")
-		(at 54.61 190.5 0)
+		(at 54.61 182.88 0)
 		(unit 1)
 		(exclude_from_sim no)
@@
 		(fields_autoplaced yes)
 		(property "Reference" "#PWR?"
-			(at 54.61 196.85 0)
+			(at 54.61 189.23 0)
 			(effects
 				(font
@@
 		)
 		(property "Value" "GND"
-			(at 54.61 195.58 0)
+			(at 54.61 187.96 0)
 			(effects
 				(font
@@
 		)
 		(property "Footprint" ""
-			(at 54.61 190.5 0)
+			(at 54.61 182.88 0)
 			(effects
 				(font
@@
 		)
 		(property "Datasheet" ""
-			(at 54.61 190.5 0)
+			(at 54.61 182.88 0)
 			(effects
 				(font
@@
 		)
 		(property "Description" "Power symbol creates a global label with name \"GND\" , ground"
-			(at 54.61 190.5 0)
-			(effects
-				(font
+			(at 54.61 182.88 0)
+			(effects
+				(font
