File: pcb/module.kicad_sch (KiCad schematic)
At the start: 19 parts, among them U3 TM1640

Commit message: use 0603 10uF caps for TM1640
Parts:
- C4: value 100uF -> 10uF; footprint Capacitor_SMD:C_1206_3216Metric -> Capacitor_SMD:C_0603_1608Metric
Changed lines of the file:
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@@
 			)
 		)
-		(property "Value" "100uF"
+		(property "Value" "10uF"
 			(at 249.174 80.772 90)
 			(effects
@@
 			)
 		)
-		(property "Footprint" "Capacitor_SMD:C_1206_3216Metric"
+		(property "Footprint" "Capacitor_SMD:C_0603_1608Metric"
 			(at 252.73 76.5048 0)
 			(effects
